File: hardware/vetus/vetus.sch (KiCad schematic (older format))
At the start: 43 parts, among them J1 anemo, J2 Conn_01x05_Male, J3 RJ45, J4 Term_sel, U1 NSI45020T1G, U10 LM4040DBZ-2.0, U11 MCP4706, U12 MCP2542FDxMF, U13 uA7805, U2 NSI45020T1G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

Commit message: Modifications mineures pour fabrication
Parts:
- U1, U2, U3, U4, U5, U6, U7, U8: symbol linear-local:NSI45020T1G -> vetus-rescue:NSI45020T1G-linear-local
- U11: symbol mcp4706:MCP4706 -> vetus-rescue:MCP4706-mcp4706
Connections:
- net CANL: now reaches J3.2, J4.4 (Pin_4), U12.6 (CANL)
- net CANH: now reaches J3.1, J4.3 (Pin_3), U12.7 (CANH)
Changed lines of the file:
@@
 NoConn ~ 3800 4150
 $Comp
-L mcp4706:MCP4706 U11
+L vetus-rescue:MCP4706-mcp4706 U11
 U 1 1 605077D8
 P 5000 6250
@@
 NoConn ~ 5400 4250
 $Comp
-L linear-local:NSI45020T1G U5
+L vetus-rescue:NSI45020T1G-linear-local U5
 U 1 1 6056B120
 P 1350 5450
@@
 	1750 5450 1850 5450
 $Comp
-L linear-local:NSI45020T1G U6
+L vetus-rescue:NSI45020T1G-linear-local U6
 U 1 1 60592D3A
 P 1350 5900
@@
 	1750 5900 1850 5900
 $Comp
-L linear-local:NSI45020T1G U7
+L vetus-rescue:NSI45020T1G-linear-local U7
 U 1 1 60596429
 P 1350 6350
@@
 	1750 6350 1850 6350
 $Comp
-L linear-local:NSI45020T1G U8
+L vetus-rescue:NSI45020T1G-linear-local U8
 U 1 1 60599C80
 P 1350 6800
@@
 	1750 6800 1850 6800
 $Comp
-L linear-local:NSI45020T1G U1
+L vetus-rescue:NSI45020T1G-linear-local U1
 U 1 1 605A2132
 P 1350 3650
@@
 	1750 3650 1850 3650
 $Comp
-L linear-local:NSI45020T1G U2
+L vetus-rescue:NSI45020T1G-linear-local U2
 U 1 1 605A2140
 P 1350 4100
@@
 	1750 4100 1850 4100
 $Comp
-L linear-local:NSI45020T1G U3
+L vetus-rescue:NSI45020T1G-linear-local U3
 U 1 1 605A214E
 P 1350 4550
@@
 	1750 4550 1850 4550
 $Comp
-L linear-local:NSI45020T1G U4
+L vetus-rescue:NSI45020T1G-linear-local U4
 U 1 1 605A215C
 P 1350 5000
@@
 Wire Wire Line
 	5300 5850 5350 5850
+Text Label 7400 4150 0    50   ~ 0
+CANH
+Text Label 7400 4250 0    50   ~ 0
+CANL
 $EndSCHEMATC
