File: hardware/capteur/capteur.kicad_pcb (KiCad board)
At the start: 2 copper layers, 125 x 65 mm, 47 parts, among them J1 Pluvio, J10 RJ45, J11 Term_sel, J12 Conn_01x05_Male, J2 Conn_01x02_Male, J3 NMEA0183 (wind), J4 Conn_01x02_Male, J5 Conn_01x02_Male, J6 Conn_01x02_Male, J7 Conn_01x03_Male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

Commit message: L'empreinte utilisée pour le connecteur RJ45 MP002453 est inversée; modification du nom utilisé pour le montrer.
Parts:
- J10: footprint local:multicomp_MP002453 -> local:multicomp_MP002453-swappedpins

Commit message: Nome les signaux SCL et SDA (pour repérage facile)
Connections:
- net Net-(J9-Pad1) renamed /SDA
- net Net-(J9-Pad2) renamed /SCL
