File: hardware/capteur/capteur.sch (KiCad schematic (older format))
At the start: 39 parts, among them J1 Pluvio, J10 RJ45, J11 Term_sel, J12 Conn_01x05_Male, J2 Conn_01x02_Male, J3 NMEA0183 (wind), J4 Conn_01x02_Male, J5 Conn_01x02_Male, J6 Conn_01x02_Male, J7 Conn_01x03_Male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

Commit message: Connect pic18's unused pins to GND
Connections:
- net GND: now also U1.4 (RA2/Vref-), U1.5 (RA3/Vref+), U1.6 (RA4)
- no-connect marks 3 -> 0
Changed lines of the file:
@@
 Wire Wire Line
 	3050 4000 2850 4000
-NoConn ~ 3800 4250
-NoConn ~ 3800 4050
 $Comp
 L Connector:Conn_01x02_Male J1
@@
 	1    0    0    -1
 $EndComp
-NoConn ~ 3800 4150
 Wire Wire Line
 	3400 5150 3800 5150
@@
 Wire Wire Line
 	5500 5150 5400 5150
+$Comp
+L power:GND #PWR?
+U 1 1 623B5C83
+P 3650 4150
+F 0 "#PWR?" H 3650 3900 50  0001 C CNN
+F 1 "GND" V 3655 4022 50  0000 R CNN
+F 2 "" H 3650 4150 50  0001 C CNN
+F 3 "" H 3650 4150 50  0001 C CNN
+	1    3650 4150
+	0    1    1    0
+$EndComp
+Wire Wire Line
+	3800 4050 3750 4050
+Wire Wire Line
+	3750 4050 3750 4150
+Wire Wire Line
+	3750 4250 3800 4250
+Wire Wire Line
+	3800 4150 3750 4150
+Connection ~ 3750 4150
+Wire Wire Line
+	3750 4150 3750 4250
+Wire Wire Line
+	3750 4150 3650 4150
 $EndSCHEMATC
