File: hardware/power/power.sch (KiCad schematic (older format))
At the start: 70 parts, among them J1 Jack-DC, J2 BATT, J3 Conn_01x05_Male, J4 RJ45, J5 RJ45, Q1 BSS123, Q2 PMOS, Q3 PMOS, Q4 BSS123, SW1 reset, U1 MC33063AP, U2 PIC18F26K80_ISS, U3 INA226, U4 MCP2542FDxMF, U5 LM358, U6 uA7805, Y1 10Mhz

Commit message: Modifications mineures pour fabrication
Parts:
- C1, C8: symbol Device:CP_Small -> power-rescue:CP_Small-Device
- Q1, Q4: symbol Device:Q_NMOS_GSD -> power-rescue:Q_NMOS_GSD-Device
- Q2, Q3: symbol Device:Q_PMOS_GSD -> power-rescue:Q_PMOS_GSD-Device
- R1, R10, R11, R12, R13, R14, R15, R16, R17, R18, R19, R2, R20, R21, R22, R23, R24, R25, R26, R27, R3, R4, R5, R6, R7, R8, R9: symbol Device:R_Small -> power-rescue:R_Small-Device
- RV1, RV2: symbol Device:R_POT_Small -> power-rescue:R_POT_Small-Device
- TH1: symbol Device:Thermistor_NTC -> power-rescue:Thermistor_NTC-Device
Changed lines of the file:
@@
 $EndComp
 $Comp
-L Device:R_Small R6
+L power-rescue:R_Small-Device R6
 U 1 1 6048396A
 P 3550 4900
@@
 $EndComp
 $Comp
-L Device:CP_Small C1
+L power-rescue:CP_Small-Device C1
 U 1 1 604A7454
 P 1950 1800
@@
 $EndComp
 $Comp
-L Device:R_Small R4
+L power-rescue:R_Small-Device R4
 U 1 1 604A7CD7
 P 2950 1500
@@
 $EndComp
 $Comp
-L Device:R_Small R5
+L power-rescue:R_Small-Device R5
 U 1 1 604A803A
 P 3250 1250
@@
 $EndComp
 $Comp
-L Device:CP_Small C8
+L power-rescue:CP_Small-Device C8
 U 1 1 604DDB56
 P 4650 1550
@@
 	4350 1150 4450 1150
 $Comp
-L Device:R_Small R8
+L power-rescue:R_Small-Device R8
 U 1 1 604F7285
 P 4450 1450
@@
 $EndComp
 $Comp
-L Device:R_Small R9
+L power-rescue:R_Small-Device R9
 U 1 1 604F76AF
 P 4450 2600
@@
 	2850 2400 3350 2400
 $Comp
-L Device:R_Small R1
+L power-rescue:R_Small-Device R1
 U 1 1 6051DA41
 P 2400 2500
@@
 $EndComp
 $Comp
-L Device:R_Small R2
+L power-rescue:R_Small-Device R2
 U 1 1 6051E81E
 P 2400 4550
@@
 $EndComp
 $Comp
-L Device:R_Small R11
+L power-rescue:R_Small-Device R11
 U 1 1 605368C3
 P 5250 2400
@@
 	5250 2500 5250 2600
 $Comp
-L Device:R_Small R15
+L power-rescue:R_Small-Device R15
 U 1 1 6057BAB5
 P 5700 2300
@@
 Connection ~ 5900 2300
 $Comp
-L Device:R_Small R16
+L power-rescue:R_Small-Device R16
 U 1 1 605AB44F
 P 5700 2500
@@
 	7950 5800 7950 5600
 $Comp
-L Device:R_Small R24
+L power-rescue:R_Small-Device R24
 U 1 1 604C17DE
 P 7700 5250
@@
 $EndComp
 $Comp
-L Device:R_Small R25
+L power-rescue:R_Small-Device R25
 U 1 1 604C17E4
 P 7700 5650
@@
 	7700 5400 7700 5550
 $Comp
-L Device:R_Small R26
+L power-rescue:R_Small-Device R26
 U 1 1 604F35AC
 P 8700 5000
@@
 $EndComp
 $Comp
-L Device:R_Small R27
+L power-rescue:R_Small-Device R27
 U 1 1 604F4DFA
 P 8800 5000
@@
 	5350 3400 5400 3400
 $Comp
-L Device:R_Small R12
+L power-rescue:R_Small-Device R12
 U 1 1 6049C932
 P 5450 3400
@@
 	4650 1150 5250 1150
 $Comp
-L Device:Q_PMOS_GSD Q3
+L power-rescue:Q_PMOS_GSD-Device Q3
 U 1 1 605084D9
 P 5350 1750
@@
 	5250 1150 5550 1150
 $Comp
-L Device:R_Small R13
+L power-rescue:R_Small-Device R13
 U 1 1 6059B2B5
 P 5550 1250
@@
 	5550 1150 8150 1150
 $Comp
-L Device:R_Small R14
+L power-rescue:R_Small-Device R14
 U 1 1 60696089
 P 5550 1850
@@
 	5500 2100 6800 2100
 $Comp
-L Device:Q_NMOS_GSD Q4
+L power-rescue:Q_NMOS_GSD-Device Q4
 U 1 1 605B5E48
 P 6450 1550
@@
 	5550 1750 5900 1750
 $Comp
-L Device:R_Small R22
+L power-rescue:R_Small-Device R22
 U 1 1 605BA937
 P 6550 1750
@@
 	6650 1550 6800 1550
 $Comp
-L Device:Thermistor_NTC TH1
+L power-rescue:Thermistor_NTC-Device TH1
 U 1 1 6094600D
 P 2600 3550
@@
 $EndComp
 $Comp
-L Device:R_Small R3
+L power-rescue:R_Small-Device R3
 U 1 1 60947665
 P 2600 3900
@@
 	2600 3750 2600 3700
 $Comp
-L Device:R_Small R20
+L power-rescue:R_Small-Device R20
 U 1 1 60A1011C
 P 6600 5850
@@
 $EndComp
 $Comp
-L Device:R_Small R18
+L power-rescue:R_Small-Device R18
 U 1 1 60A1092C
 P 6350 5850
@@
 	6350 5500 5400 5500
 $Comp
-L Device:R_Small R17
+L power-rescue:R_Small-Device R17
 U 1 1 60A5DBF1
 P 5950 4950
@@
 $EndComp
 $Comp
-L Device:R_Small R19
+L power-rescue:R_Small-Device R19
 U 1 1 60A6033F
 P 6150 4750
@@
 $EndComp
 $Comp
-L Device:R_Small R21
+L power-rescue:R_Small-Device R21
 U 1 1 60A60988
 P 6400 4950
@@
 $EndComp
 $Comp
-L Device:R_Small R23
+L power-rescue:R_Small-Device R23
 U 1 1 60A610DF
 P 6600 4750
@@
 NoConn ~ 1800 1800
 $Comp
-L Device:Q_PMOS_GSD Q2
+L power-rescue:Q_PMOS_GSD-Device Q2
 U 1 1 604F9FE0
 P 5350 1350
@@
 	4450 1550 4450 2200
 $Comp
-L Device:R_POT_Small RV2
+L power-rescue:R_POT_Small-Device RV2
 U 1 1 60652FE8
 P 4450 2350
@@
 NoConn ~ 4450 2250
 $Comp
-L Device:R_Small R7
+L power-rescue:R_Small-Device R7
 U 1 1 6069273B
 P 4100 2600
@@
 $EndComp
 $Comp
-L Device:R_POT_Small RV1
+L power-rescue:R_POT_Small-Device RV1
 U 1 1 60692B9C
 P 4100 2350
@@
 	4100 2700 4100 2750
 $Comp
-L Device:Q_NMOS_GSD Q1
+L power-rescue:Q_NMOS_GSD-Device Q1
 U 1 1 6076683C
 P 4200 2950
@@
 Connection ~ 4650 2800
 $Comp
-L Device:R_Small R10
+L power-rescue:R_Small-Device R10
 U 1 1 607781B9
 P 4450 3050

Commit message: Ajout référence NTC
Parts:
- TH1: symbol power-rescue:Thermistor_NTC-Device -> Device:Thermistor_NTC; P/N (none) -> ND06P00103K
Changed lines of the file:
@@
 	6650 1550 6800 1550
 $Comp
-L power-rescue:Thermistor_NTC-Device TH1
+L Device:Thermistor_NTC TH1
 U 1 1 6094600D
 P 2600 3550
@@
 F 2 "Connector_PinHeader_2.54mm:PinHeader_1x02_P2.54mm_Vertical" H 2600 3600 50  0001 C CNN
 F 3 "~" H 2600 3600 50  0001 C CNN
+F 4 "ND06P00103K" H 2600 3550 50  0001 C CNN "P/N"
 	1    2600 3550
 	1    0    0    -1
