File: hardware/centrale/keys.kicad_pcb (KiCad board)
At the start: 2 copper layers, 34 x 38.5 mm, 15 parts, among them J1 LRADC, J2 GND, J3 BME280, J4 SDA, J5 SCL, J6 +3.3V, SW1 Left, SW2 Up, SW3 Down, SW4 Right

Commit message: Add 5mm margin around PCBs
Other:
- board size 34 x 38.5 mm -> 44 x 48.5 mm

Commit message: clips are not strong enough, so remplace with a screw for PCB
Parts:
- added REF**: MountingHole_3.2mm_M3, MountingHole:MountingHole_3.2mm_M3, F.Cu at (102.5, 102.5)
- moved R4 15.7 mm to (94.5, 110.5), turned to 270 degrees
- moved R1 12.0 mm to (88.5, 94.0), turned to 270 degrees
- moved R2 10.9 mm to (94.5, 94.0), turned to 90 degrees
- moved R3 10.2 mm to (92.2, 110.5), turned to 90 degrees
- moved R5 7.54 mm to (113.0, 108.2)
- moved J2 6.10 mm to (88.0, 110.8)
- moved J4 3.00 mm to (93.6, 87.4)
- moved J5 3.00 mm to (93.6, 90.6)
Routing:
- net Net-(R2-Pad1): track 13.0 -> 35.9 mm
- net Net-(R4-Pad1): track 11.7 -> 28.1 mm
- net /LRADC: track 8.20 -> 3.13 mm
- net Net-(R1-Pad2): track 15.4 -> 10.4 mm
- net Net-(R3-Pad1): track 6.73 -> 2.25 mm
- net /SDA: track 12.6 -> 9.24 mm
- net /SCL: track 16.6 -> 13.3 mm
- net Net-(R1-Pad1): track 14.1 -> 16.5 mm
