File: hardware/centrale/centrale.kicad_sch (KiCad schematic)
At the start: 36 parts, among them U1 MCP7940N-xSN

Commit message: Name CANH and CANL nets
Parts:
- +5V1: value (none) -> 5V_LIME2; footprint (none) -> local:MC24356
- BT1: value (none) -> CR2032; footprint (none) -> local:1066
- C1, C2: value (none) -> 10pF; footprint (none) -> Capacitor_SMD:C_0603_1608Metric_Pad1.08x0.95mm_HandSolder
- C10, C8, C9: value (none) -> 1uF16V; footprint (none) -> Capacitor_SMD:C_0805_2012Metric_Pad1.18x1.45mm_HandSolder
- C11, C5: value (none) -> 100nF6.3V; footprint (none) -> Capacitor_SMD:C_0805_2012Metric_Pad1.18x1.45mm_HandSolder
- C12: value (none) -> 10pf; footprint (none) -> Capacitor_SMD:C_0603_1608Metric_Pad1.08x0.95mm_HandSolder
- C13, C14: value (none) -> 22µF6.3V; footprint (none) -> Capacitor_SMD:C_1210_3225Metric_Pad1.33x2.70mm_HandSolder
- C15, C16: value (none) -> 100nF; footprint (none) -> Capacitor_SMD:C_0805_2012Metric_Pad1.18x1.45mm_HandSolder
- C3: value (none) -> 6.8nF; footprint (none) -> Capacitor_SMD:C_0603_1608Metric_Pad1.08x0.95mm_HandSolder
- C4: value (none) -> 1µF6.3v; footprint (none) -> Capacitor_SMD:C_0805_2012Metric_Pad1.18x1.45mm_HandSolder
- C6: value (none) -> 1uF25V; footprint (none) -> Capacitor_SMD:C_0805_2012Metric_Pad1.18x1.45mm_HandSolder
- C7: value (none) -> 10µF25V; footprint (none) -> Capacitor_SMD:C_1210_3225Metric_Pad1.33x2.70mm_HandSolder
- D1: value (none) -> SMBJ16A; footprint (none) -> Diode_SMD:D_SMB_Handsoldering
- J1: value (none) -> MDCOG240128B6W; footprint (none) -> local:multicomp505110-2691
- J2: value (none) -> Conn_BME280; footprint (none) -> jst:JST_S6B-ZR-SM4A-TF(LF)(SN)
- J3: value (none) -> CONN_BME280_2; footprint (none) -> te:CONN-TE-MICROMATCH-5X2-PTH-BOSS
- J4: value (none) -> RJ45; footprint (none) -> Connector_RJ:RJ45_Amphenol_54602-x08_Horizontal
- J5: value (none) -> Term_sel; footprint (none) -> Connector_PinHeader_2.54mm:PinHeader_2x03_P2.54mm_Vertical
- L1: value (none) -> 4.7µH; footprint (none) -> local:L_TT_7.3x6.8
- Q1: value (none) -> BSS123; footprint (none) -> Package_TO_SOT_SMD:SOT-23
- R1, R3: value (none) -> 10K; footprint (none) -> Resistor_SMD:R_1206_3216Metric_Pad1.30x1.75mm_HandSolder
- R2: value (none) -> 4K7; footprint (none) -> Resistor_SMD:R_0805_2012Metric_Pad1.20x1.40mm_HandSolder
- R4: value (none) -> 56K; footprint (none) -> Resistor_SMD:R_0805_2012Metric_Pad1.20x1.40mm_HandSolder
- R5: value (none) -> 47K; footprint (none) -> Resistor_SMD:R_0805_2012Metric_Pad1.20x1.40mm_HandSolder
- R6: value (none) -> 100; footprint (none) -> Resistor_SMD:R_0805_2012Metric_Pad1.20x1.40mm_HandSolder
- U2: value (none) -> TPS54228; footprint (none) -> Package_SO:SOIC-8-1EP_3.9x4.9mm_P1.27mm_EP2.41x3.3mm
- U3: value (none) -> TLE9250V; footprint (none) -> Package_SO:SOIC-8_3.9x4.9mm_P1.27mm
- Y1: value (none) -> 32.768Khz; footprint (none) -> local:CMR200T
Connections:
- net CANL: now reaches J4.2, J5.3 (Pin_3), U3.6 (CANL)
- net CANH: now reaches J4.1, J5.4 (Pin_4), U3.7 (CANH)
