File: hardware/centrale/lime2.kicad_sch (KiCad schematic)
At the start: 2 parts

Commit message: Name CANH and CANL nets
Parts:
- GPIO-1, GPIO-3: renamed from GPIO-?; value (none) -> FL40YA-V36P-2X20-LF; footprint (none) -> A20_OLIMEXINO_LIME2_SHIELD:A20_OLIMEXINO_LIME2_SHIELD_1-YA-V36P-2X20-LF
Changed lines of the file:
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@@
   (symbol (lib_id "centrale-rescue:FL40YA-V36P-2X20-LF") (at 109.22 53.34 0) (mirror x) (unit 1)
     (in_bom yes) (on_board yes)
-    (property "Reference" "GPIO-?" (id 0) (at 105.41 22.86 0)
-      (effects (font (size 1.27 1.27)) (justify left bottom))
-    )
-    (property "Value" "" (id 1) (at 97.79 80.01 0)
-      (effects (font (size 1.27 1.27)) (justify left bottom))
-    )
-    (property "Footprint" "" (id 2) (at 109.22 57.15 0)
+    (property "Reference" "GPIO-1" (id 0) (at 105.41 22.86 0)
+      (effects (font (size 1.27 1.27)) (justify left bottom))
+    )
+    (property "Value" "FL40YA-V36P-2X20-LF" (id 1) (at 97.79 80.01 0)
+      (effects (font (size 1.27 1.27)) (justify left bottom))
+    )
+    (property "Footprint" "A20_OLIMEXINO_LIME2_SHIELD:A20_OLIMEXINO_LIME2_SHIELD_1-YA-V36P-2X20-LF" (id 2) (at 109.22 57.15 0)
       (effects (font (size 1.27 1.27)) hide)
     )
@@
   (symbol (lib_id "centrale-rescue:GND") (at 184.15 27.94 90) (unit 1)
     (in_bom yes) (on_board yes)
-    (property "Reference" "#PWR?" (id 0) (at 184.15 27.94 0)
-      (effects (font (size 0.762 0.762)) hide)
-    )
-    (property "Value" "" (id 1) (at 185.928 27.94 0)
+    (property "Reference" "#PWR06" (id 0) (at 184.15 27.94 0)
+      (effects (font (size 0.762 0.762)) hide)
+    )
+    (property "Value" "GND" (id 1) (at 185.928 27.94 0)
       (effects (font (size 0.762 0.762)) hide)
     )
@@
   (symbol (lib_id "centrale-rescue:GNDPWR") (at 186.69 30.48 90) (unit 1)
     (in_bom yes) (on_board yes)
-    (property "Reference" "#PWR?" (id 0) (at 185.42 30.48 0)
+    (property "Reference" "#PWR05" (id 0) (at 185.42 30.48 0)
       (effects (font (size 1.016 1.016)) hide)
     )
-    (property "Value" "" (id 1) (at 189.23 31.75 0)
+    (property "Value" "GNDPWR" (id 1) (at 189.23 31.75 0)
       (effects (font (size 1.016 1.016)))
     )
@@
   (symbol (lib_id "centrale-rescue:FL40YA-V36P-2X20-LF") (at 184.15 190.5 0) (mirror x) (unit 1)
     (in_bom yes) (on_board yes)
-    (property "Reference" "GPIO-?" (id 0) (at 180.34 160.02 0)
-      (effects (font (size 1.27 1.27)) (justify left bottom))
-    )
-    (property "Value" "" (id 1) (at 172.72 217.17 0)
-      (effects (font (size 1.27 1.27)) (justify left bottom))
-    )
-    (property "Footprint" "" (id 2) (at 184.15 194.31 0)
+    (property "Reference" "GPIO-3" (id 0) (at 180.34 160.02 0)
+      (effects (font (size 1.27 1.27)) (justify left bottom))
+    )
+    (property "Value" "FL40YA-V36P-2X20-LF" (id 1) (at 172.72 217.17 0)
+      (effects (font (size 1.27 1.27)) (justify left bottom))
+    )
+    (property "Footprint" "A20_OLIMEXINO_LIME2_SHIELD:A20_OLIMEXINO_LIME2_SHIELD_1-YA-V36P-2X20-LF" (id 2) (at 184.15 194.31 0)
       (effects (font (size 1.27 1.27)) hide)
     )
@@
   (symbol (lib_id "centrale-rescue:GND") (at 215.9 165.1 90) (unit 1)
     (in_bom yes) (on_board yes)
-    (property "Reference" "#PWR?" (id 0) (at 215.9 165.1 0)
-      (effects (font (size 0.762 0.762)) hide)
-    )
-    (property "Value" "" (id 1) (at 217.678 165.1 0)
+    (property "Reference" "#PWR07" (id 0) (at 215.9 165.1 0)
+      (effects (font (size 0.762 0.762)) hide)
+    )
+    (property "Value" "GND" (id 1) (at 217.678 165.1 0)
       (effects (font (size 0.762 0.762)) hide)
     )
@@
       (effects (font (size 1.27 1.27)) hide)
     )
-    (property "Value" "" (id 1) (at 140.081 155.6258 0))
+    (property "Value" "+3.3V" (id 1) (at 140.081 155.6258 0))
     (property "Footprint" "" (id 2) (at 139.7 160.02 0)
       (effects (font (size 1.27 1.27)) hide)
@@
       (effects (font (size 1.27 1.27)) hide)
     )
-    (property "Value" "" (id 1) (at 145.161 155.6258 0))
+    (property "Value" "+5V" (id 1) (at 145.161 155.6258 0))
     (property "Footprint" "" (id 2) (at 144.78 160.02 0)
       (effects (font (size 1.27 1.27)) hide)
@@
       (effects (font (size 1.27 1.27)) hide)
     )
-    (property "Value" "" (id 1) (at 70.231 18.4658 0))
+    (property "Value" "+5V" (id 1) (at 70.231 18.4658 0))
     (property "Footprint" "" (id 2) (at 69.85 22.86 0)
       (effects (font (size 1.27 1.27)) hide)
@@
       (effects (font (size 1.27 1.27)) hide)
     )
-    (property "Value" "" (id 1) (at 65.151 18.4658 0))
+    (property "Value" "+3.3V" (id 1) (at 65.151 18.4658 0))
     (property "Footprint" "" (id 2) (at 64.77 22.86 0)
       (effects (font (size 1.27 1.27)) hide)
